Commit message: ros2 control in simulation working properly (tuning of physics parameters might be needed)

File: rusty_rover_ws/src/rusty_description/urdf/include/base.urdf.xacro (robot description, xacro)
@@ -56,14 +56,9 @@
   - origin [block]: origin, position and orientation of the link;
 -->
-  <xacro:macro name="footprint"
-               params="wheel_props">
-    <!-- Base-Footprint -->
-    <!-- base_footprint is a fictitious link(frame) that is on the ground right below base_link origin -->
+<xacro:macro name="footprint" params="wheel_props">
     <link name="base_footprint" />
-    <!-- Joint to connect base_footprint with base_link -->
     <joint name="base_footprint_joint" type="fixed">
-      <parent link="base_link"/>
-      <child link="base_footprint" />
-      <origin xyz="0 0 ${-(wheel_props['radius'] - wheel_props['z_offset'])}" rpy="0 0 0" />
+      <parent link="base_footprint"/> <child link="base_link" />
+      <origin xyz="0 0 ${(wheel_props['radius'] - wheel_props['z_offset'])}" rpy="0 0 0" />
     </joint>
   </xacro:macro>

File: rusty_rover_ws/src/rusty_description/urdf/include/rusty_control.urdf.xacro (robot description, xacro)
@@ -2,45 +2,34 @@
 <robot xmlns:xacro="http://www.ros.org/wiki/xacro">
   <xacro:macro name="rusty_ros2_control" params="sim_mode">
-    <xacro:if value="${sim_mode}">
-        <ros2_control name="GazeboSimSystem" type="system">
-            <hardware>
-                <plugin>gz_ros2_control/GazeboSimSystem</plugin>
-            </hardware>
-            <joint name="left_wheel_joint">
-                <command_interface name="velocity"/>
-                <state_interface name="velocity" />
-            </joint>
-            <joint name="right_wheel_joint">
-                <command_interface name="velocity"/>
-                <state_interface name="velocity" />
-            </joint>
-        </ros2_control>
-    </xacro:if>
-    <xacro:unless value="${sim_mode}">
-        <ros2_control name="RealRobot" type="system">
-            <hardware>
-                <plugin>rusty_control/RustySystemHardware</plugin>
-                <param name="pin_enable_0">8</param>
-                <param name="pin_pos_0">9</param>
-                <param name="pin_neg_0">10</param>
-                <param name="pin_enable_1">13</param>
-                <param name="pin_pos_1">12</param>
-                <param name="pin_neg_1">11</param>
-            </hardware>
-            <joint name="left_wheel_joint">
-                <command_interface name="velocity"/>
-                <state_interface name="velocity" />
-            </joint>
-            <joint name="right_wheel_joint">
-                <command_interface name="velocity"/>
-                <state_interface name="velocity" />
-            </joint>
-        </ros2_control>
-    </xacro:unless>
-    <gazebo>
-        <plugin filename="libgz_ros2_control-system.so" name="gz_ros2_control::GazeboSimROS2ControlPlugin">
-            <parameters>$(find rusty_control)/config/controller.yaml</parameters>
-        </plugin>
-    </gazebo>
+    <ros2_control name="RustyControlSystem" type="system">
+      <hardware>
+        <xacro:if value="${sim_mode}">
+          <plugin>gz_ros2_control/GazeboSimSystem</plugin>
+        </xacro:if>
+        <xacro:unless value="${sim_mode}">
+          <plugin>rusty_control/RustySystemHardware</plugin>
+          <param name="pin_enable_0">8</param>
+          <param name="pin_pos_0">9</param>
+          <param name="pin_neg_0">10</param>
+          <param name="pin_enable_1">13</param>
+          <param name="pin_pos_1">12</param>
+          <param name="pin_neg_1">11</param>
+        </xacro:unless>
+      </hardware>
+      <joint name="left_wheel_joint">
+        <command_interface name="velocity">
+          <param name="min">-10</param>
+          <param name="max">10</param>
+        </command_interface>
+        <state_interface name="position"/> <state_interface name="velocity"/>
+      </joint>
+      <joint name="right_wheel_joint">
+        <command_interface name="velocity">
+          <param name="min">-10</param>
+          <param name="max">10</param>
+        </command_interface>
+        <state_interface name="position"/> <state_interface name="velocity"/>
+      </joint>
+    </ros2_control>
   </xacro:macro>
 </robot>

File: rusty_rover_ws/src/rusty_description/urdf/rusty.urdf.xacro (robot description, xacro)
@@ -45,3 +45,12 @@
   <!-- ros2_control -->
   <xacro:rusty_ros2_control sim_mode="$(arg sim_mode)" />
+  <!-- Gazebo plugin for ros2 control -->
+  <gazebo>
+    <plugin name="gz_ros2_control::GazeboSimROS2ControlPlugin" filename="libgz_ros2_control-system.so">
+      <parameters>$(find rusty_control)/config/controller.yaml</parameters>
+      <ros>
+        <use_sim_time>true</use_sim_time>
+      </ros>
+    </plugin>
+  </gazebo>
 </robot>
