Commit message: Caster wheel witout friction + kinematic adjustments in controller params

File: rusty_rover_ws/src/rusty_description/urdf/include/caster_wheel.urdf.xacro (robot description, xacro)
@@ -58,4 +58,13 @@
       <dynamics damping="0.01" friction="0.0"/>
     </joint>
+    <!-- Gazebo: ultra-low friction on the ball -->
+    <gazebo reference="caster_base_link">
+      <mu1>0.0</mu1>
+      <mu2>0.0</mu2>
+      <kp>1000000.0</kp>
+      <kd>1.0</kd>
+      <minDepth>0.001</minDepth>
+      <material>Gazebo/Black</material>
+    </gazebo>
   </xacro:macro>
 </robot>
